File: BTMessBox/BTMessBox.kicad_pcb (KiCad board)
At the start: 2 copper layers, 77.5 x 108 mm, 73 parts, among them J1 JST-Bu, J2 JST-Bu, J3 JST-Bu, J4 JST-Bu, J5 JST-Bu, J6 JST-Bu, J7 JST-BU, U1 MCP6044, U2 MCP6044, U3 MCP3208-BI/SL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

Commit message: Anpassungen
Parts:
- added R33: 10k, Resistor_SMD:R_0805_2012Metric_Pad1.20x1.40mm_HandSolder, F.Cu at (47.0, 118.0)
- added R34: 10k, Resistor_SMD:R_0805_2012Metric_Pad1.20x1.40mm_HandSolder, F.Cu at (46.0, 122.0)
- R25, R26, R27, R28, R29, R30: value 140k -> 150k
Connections:
- U2 pad 10: GND -> Net-(U2C-+)
- U2 pad 12: GND -> Net-(U2C-+)
Routing:
- net Net-(U2C-+): track 0.00 -> 19.7 mm
- net GND: track 566.6 -> 558.5 mm
- net +3.3V: track 243.7 -> 245.2 mm
- net ADC0: track 39.3 -> 37.9 mm
