File: BTMessBox/BTMessBox.kicad_sch (KiCad schematic)
At the start: 73 parts, among them J1 JST-Bu, J2 JST-Bu, J3 JST-Bu, J4 JST-Bu, J5 JST-Bu, J6 JST-Bu, J7 JST-BU, U1 MCP6044, U2 MCP6044, U3 MCP3208-BI/SL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

Commit message: Anpassungen
Parts:
- added R33, R34: 10k, Resistor_SMD:R_0805_2012Metric_Pad1.20x1.40mm_HandSolder, symbol Device:R
- R25, R26, R27, R28, R29, R30: value 140k -> 150k
Connections:
- net +3.3V: now also R33.1
- net GND: now also R34.2; no longer U2.10 (+), U2.12 (+)
- new net: R33.2, R34.1, U2.10 (+), U2.12 (+)
Other:
- note added: "6-Kanal Sensor f. Strom- und Spannungsausgang"
- note added: "AD-Wandler"
- note added: "ESP-32 Mikroprozessor"
- note added: "Referenzspannungsquelle"
- note added: "Signaleingänge"
- note added: "Signalverstärkung"
- note added: "Spannungsversorgung"
- note added: "Spannungsversorgung OP"
- note added: "Ungenutze OP"
- note removed: "7-Kanal Sensor f. Strom- und Spannungsausgang"
- moved on the sheet: C1, C10, C11, C12, C13, C14, C15, C16, C17, C18, C19, C2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
